Commit message: Working commit

File: src/sb_gazebo/urdf/macros.xacro (robot description, xacro)
@@ -108,5 +108,5 @@
   <axis xyz="0 1 0" rpy="0 0 0" />
   <limit effort="100" velocity="100"/>
-  <joint_properties damping="1.0" friction="1.0"/>
+  <joint_properties damping="2.0" friction="1.0"/>
   <hardwareInterface>EffortJointInterface</hardwareInterface>
 </joint>

File: src/sb_gazebo/urdf/oaken.xacro (robot description, xacro)
@@ -8,5 +8,5 @@
 <xacro:property name="chassis_width" value="0.85" />
 <xacro:property name="chassis_height" value="0.35" />
-<xacro:property name="chassis_mass" value="30" />
+<xacro:property name="chassis_mass" value="50" />
 <xacro:property name="chassis_elevation" value="0.1" />
 <xacro:property name="tower_height" value="0.9"/>
@@ -16,5 +16,5 @@
 <xacro:property name="wheel_width" value="0.15" />
 <xacro:property name="wheel_displace" value="0.25" />
-<xacro:property name="wheel_mass" value="1" />
+<xacro:property name="wheel_mass" value="3" />
 <xacro:property name="camera_size" value="0.05" />
 <xacro:property name="camera_mass" value="0.1" />
